File: G030F6P6_test/G030F6P6_test.kicad_sch (KiCad schematic)
At the start: 28 parts, among them J1 Conn_01x10_Female, J2 Conn_01x10_Female, J3 USB_C_Receptacle_USB2.0, J5 Conn_01x05_Female, U1 CH343P, U2 STM32G030FxP, U3 XC6206P332MR

Commit message: 送交打樣
Parts:
- C1, C2, C3, C4, C5: value 0.1uF -> (none); footprint Capacitor_SMD:C_0805_2012Metric -> (none); LCSC C1711 -> C72038
- J1, J2: value Conn_01x10_Female -> (none); footprint Connector_PinHeader_2.54mm:PinHeader_1x10_P2.54mm_Vertical -> (none)
- J4: now left out of the parts list
- J5: value Conn_01x05_Female -> (none); footprint Connector_PinHeader_2.54mm:PinHeader_1x05_P2.54mm_Vertical -> (none); now in the parts list
Changed lines of the file:
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@@
       (effects (font (size 1.27 1.27)) (justify left))
     )
-    (property "Value" "0.1uF" (id 1) (at 223.901 53.219 0)
-      (effects (font (size 1.27 1.27)) (justify left))
-    )
-    (property "Footprint" "Capacitor_SMD:C_0805_2012Metric" (id 2) (at 224.4852 54.61 0)
+    (property "Value" "" (id 1) (at 223.901 53.219 0)
+      (effects (font (size 1.27 1.27)) (justify left))
+    )
+    (property "Footprint" "" (id 2) (at 224.4852 54.61 0)
       (effects (font (size 1.27 1.27)) hide)
     )
@@
       (effects (font (size 1.27 1.27)) hide)
     )
-    (property "LCSC" "C1711" (id 4) (at 223.52 50.8 0)
+    (property "LCSC" "C72038" (id 4) (at 223.52 50.8 0)
       (effects (font (size 1.27 1.27)) hide)
     )
@@
       (effects (font (size 1.27 1.27)) (justify left))
     )
-    (property "Value" "0.1uF" (id 1) (at 195.961 53.219 0)
-      (effects (font (size 1.27 1.27)) (justify left))
-    )
-    (property "Footprint" "Capacitor_SMD:C_0805_2012Metric" (id 2) (at 196.5452 54.61 0)
+    (property "Value" "" (id 1) (at 195.961 53.219 0)
+      (effects (font (size 1.27 1.27)) (justify left))
+    )
+    (property "Footprint" "" (id 2) (at 196.5452 54.61 0)
       (effects (font (size 1.27 1.27)) hide)
     )
@@
       (effects (font (size 1.27 1.27)) hide)
     )
-    (property "LCSC" "C1711" (id 4) (at 195.58 50.8 0)
+    (property "LCSC" "C72038" (id 4) (at 195.58 50.8 0)
       (effects (font (size 1.27 1.27)) hide)
     )
@@
       (effects (font (size 1.27 1.27)) (justify left))
     )
-    (property "Value" "0.1uF" (id 1) (at 146.431 181.489 0)
-      (effects (font (size 1.27 1.27)) (justify left))
-    )
-    (property "Footprint" "Capacitor_SMD:C_0805_2012Metric" (id 2) (at 147.0152 182.88 0)
+    (property "Value" "" (id 1) (at 146.431 181.489 0)
+      (effects (font (size 1.27 1.27)) (justify left))
+    )
+    (property "Footprint" "" (id 2) (at 147.0152 182.88 0)
       (effects (font (size 1.27 1.27)) hide)
     )
@@
       (effects (font (size 1.27 1.27)) hide)
     )
-    (property "LCSC" "C1711" (id 4) (at 146.05 179.07 0)
+    (property "LCSC" "C72038" (id 4) (at 146.05 179.07 0)
       (effects (font (size 1.27 1.27)) hide)
     )
@@
   )
   (symbol (lib_id "Connector:Conn_01x05_Female") (at 270.51 106.045 0) (unit 1)
-    (in_bom no) (on_board yes)
+    (in_bom yes) (on_board yes)
     (property "Reference" "J5" (id 0) (at 269.24 97.79 0)
       (effects (font (size 1.27 1.27)) (justify left))
     )
-    (property "Value" "Conn_01x05_Female" (id 1) (at 256.54 113.03 0)
-      (effects (font (size 1.27 1.27)) (justify left))
-    )
-    (property "Footprint" "Connector_PinHeader_2.54mm:PinHeader_1x05_P2.54mm_Vertical" (id 2) (at 270.51 106.045 0)
+    (property "Value" "" (id 1) (at 256.54 113.03 0)
+      (effects (font (size 1.27 1.27)) (justify left))
+    )
+    (property "Footprint" "" (id 2) (at 270.51 106.045 0)
       (effects (font (size 1.27 1.27)) hide)
     )
@@
   )
   (symbol (lib_id "Connector_Generic:Conn_02x02_Odd_Even") (at 160.02 143.51 0) (unit 1)
-    (in_bom yes) (on_board yes) (fields_autoplaced)
+    (in_bom no) (on_board yes) (fields_autoplaced)
     (property "Reference" "J4" (id 0) (at 161.29 137.16 0))
     (property "Value" "" (id 1) (at 161.29 139.7 0))
@@
       (effects (font (size 1.27 1.27)) (justify left))
     )
-    (property "Value" "0.1uF" (id 1) (at 60.071 43.059 0)
-      (effects (font (size 1.27 1.27)) (justify left))
-    )
-    (property "Footprint" "Capacitor_SMD:C_0805_2012Metric" (id 2) (at 60.6552 44.45 0)
+    (property "Value" "" (id 1) (at 60.071 43.059 0)
+      (effects (font (size 1.27 1.27)) (justify left))
+    )
+    (property "Footprint" "" (id 2) (at 60.6552 44.45 0)
       (effects (font (size 1.27 1.27)) hide)
     )
@@
       (effects (font (size 1.27 1.27)) hide)
     )
-    (property "LCSC" "C1711" (id 4) (at 59.69 40.64 0)
+    (property "LCSC" "C72038" (id 4) (at 59.69 40.64 0)
       (effects (font (size 1.27 1.27)) hide)
     )
@@
       (effects (font (size 1.27 1.27)) (justify left))
     )
-    (property "Value" "Conn_01x10_Female" (id 1) (at 126.365 175.8949 0)
+    (property "Value" "" (id 1) (at 126.365 175.8949 0)
       (effects (font (size 1.27 1.27)) (justify left) hide)
     )
-    (property "Footprint" "Connector_PinHeader_2.54mm:PinHeader_1x10_P2.54mm_Vertical" (id 2) (at 124.46 173.355 0)
+    (property "Footprint" "" (id 2) (at 124.46 173.355 0)
       (effects (font (size 1.27 1.27)) hide)
     )
@@
       (effects (font (size 1.27 1.27)) (justify left))
     )
-    (property "Value" "Conn_01x10_Female" (id 1) (at 36.195 176.5299 0)
+    (property "Value" "" (id 1) (at 36.195 176.5299 0)
       (effects (font (size 1.27 1.27)) (justify left) hide)
     )
-    (property "Footprint" "Connector_PinHeader_2.54mm:PinHeader_1x10_P2.54mm_Vertical" (id 2) (at 34.29 173.99 0)
+    (property "Footprint" "" (id 2) (at 34.29 173.99 0)
       (effects (font (size 1.27 1.27)) hide)
     )
@@
       (effects (font (size 1.27 1.27)) (justify left))
     )
-    (property "Value" "0.1uF" (id 1) (at 37.211 68.459 0)
-      (effects (font (size 1.27 1.27)) (justify left))
-    )
-    (property "Footprint" "Capacitor_SMD:C_0805_2012Metric" (id 2) (at 37.7952 69.85 0)
+    (property "Value" "" (id 1) (at 37.211 68.459 0)
+      (effects (font (size 1.27 1.27)) (justify left))
+    )
+    (property "Footprint" "" (id 2) (at 37.7952 69.85 0)
       (effects (font (size 1.27 1.27)) hide)
     )
@@
       (effects (font (size 1.27 1.27)) hide)
     )
-    (property "LCSC" "C1711" (id 4) (at 36.83 66.04 0)
-      (effects (font (size 1.27 1.27)) hide)
-    )
+    (property "LCSC" "C72038" (id 4) (at 36.83 66.04 0)
+      (effects (font (size 1.27 1.27)) hide)
+    )
