File: G030F6P6_test/G030F6P6_test.kicad_pcb (KiCad board)
At the start: 2 copper layers, 22.9 x 49.1 mm, 29 parts, among them J1 Conn_01x10_Female, J2 Conn_01x10_Female, J3 USB_C_Receptacle_USB2.0, J4 Conn_02x02_Odd_Even, J5 Conn_01x05_Female, U1 CH343P, U2 STM32G030FxP, U3 XC6206P332MR

Commit message: jlcpcb 打樣
Parts:
- moved R2 16.4 mm to (121.2, 58.0)
- moved R3 15.0 mm to (123.4, 58.0), turned to -90 degrees
- moved REF** 0.51 mm to (138.6, 63.5)
Routing:
- net /CC1: track 7.91 -> 13.1 mm
- net +3V3: track 56.3 -> 58.8 mm
- net /CC2: track 10.9 -> 12.4 mm
- net VBUS: track 30.9 -> 31.9 mm
- net /TXD: track 15.7 -> 16.3 mm
- net GND: track 1.20 -> 1.62 mm, vias 3 -> 17
